File: USB.sch (KiCad schematic (older format))
At the start: 10 parts

Commit message: corrected CAN schematic
Parts:
- C10: renamed from C?; footprint (none) -> Capacitor_SMD:C_0805_2012Metric; Description (none) -> 10uF ±10% 10V X5R 0805 Multilayer Ceramic Capacitors MLCC; Manufacturer (none) -> Samsung Electro-Mechanics; Mount (none) -> MOUNT; MountType (none) -> SMD; PartNumber (none) -> CL21A106KPFNNNE
- C11, C12: renamed from C?; footprint (none) -> Capacitor_SMD:C_0603_1608Metric; Description (none) -> 47pF ±10% 50V C0G 0603 Multilayer Ceramic Capacitors; Manufacturer (none) -> Samsung Electro-Mechanics; Mount (none) -> MOUNT; MountType (none) -> SMD; PartNumber (none) -> CL10C470KB8NNNC
- J4: renamed from J?; Manufacturer (none) -> -; Mount (none) -> MOUNT; MountType (none) -> SMD
- R11: renamed from R?; Description (none) -> 4.7kΩ ±1% 0.1W ±100ppm/℃ 0603 Chip Resistor - Surface Mount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; Manufacturer (none) -> YAGEO; Mount (none) -> MOUNT; MountType (none) -> SMD; PartNumber (none) -> RC0603FR-074K7L
- R12, R13, R14, R15: renamed from R?; Manufacturer (none) -> -; Mount (none) -> MOUNT; MountType (none) -> SMD
- U2: renamed from U?; Description (none) -> Unidirectional 5.25V 6V 17V 5A SOT-23-6 Diodes; Manufacturer (none) -> ST Microelectronics; Mount (none) -> MOUNT; MountType (none) -> SMD; PartNumber (none) -> USBLC6-2SC6
Changed lines of the file:
@@
 P 1650 2600
 AR Path="/6008501D/600878DC" Ref="J?"  Part="1"
-AR Path="/60084FF3/600A49FC/600878DC" Ref="J?"  Part="1"
-F 0 "J?" H 1500 2950 50  0000 C CNN
+AR Path="/60084FF3/600A49FC/600878DC" Ref="J4"  Part="1"
+F 0 "J4" H 1500 2950 50  0000 C CNN
 F 1 "USB_B_Micro" H 1707 2976 50  0001 C CNN
 F 2 "Connector_USB:USB_Micro-B_GCT_USB3076-30-A" H 1800 2550 50  0001 C CNN
 F 3 "~" H 1800 2550 50  0001 C CNN
+F 4 "MOUNT" H 1650 2600 50  0001 C CNN "Mount"
+F 5 "SMD" H 1650 2600 50  0001 C CNN "MountType"
+F 6 "-" H 1650 2600 50  0001 C CNN "Manufacturer"
 	1    1650 2600
 	1    0    0    -1
@@
 P 3750 2650
 AR Path="/6008501D/6008874E" Ref="U?"  Part="1"
-AR Path="/60084FF3/600A49FC/6008874E" Ref="U?"  Part="1"
-F 0 "U?" V 4000 3000 50  0000 L CNN
+AR Path="/60084FF3/600A49FC/6008874E" Ref="U2"  Part="1"
+F 0 "U2" V 4000 3000 50  0000 L CNN
 F 1 "USBLC6-2SC6" V 4100 3000 50  0000 L CNN
 F 2 "Package_TO_SOT_SMD:SOT-23-6" H 3000 3050 50  0001 C CNN
 F 3 "http://www2.st.com/resource/en/datasheet/CD00050750.pdf" H 3950 3000 50  0001 C CNN
+F 4 "MOUNT" H 3750 2650 50  0001 C CNN "Mount"
+F 5 "SMD" H 3750 2650 50  0001 C CNN "MountType"
+F 6 "ST Microelectronics" H 3750 2650 50  0001 C CNN "Manufacturer"
+F 7 "USBLC6-2SC6" H 3750 2650 50  0001 C CNN "PartNumber"
+F 8 "Unidirectional 5.25V 6V 17V 5A SOT-23-6 Diodes" H 3750 2650 50  0001 C CNN "Description"
 	1    3750 2650
 	0    1    1    0
@@
 P 1650 3100
 AR Path="/6008501D/6008C2BE" Ref="#PWR?"  Part="1"
-AR Path="/60084FF3/600A49FC/6008C2BE" Ref="#PWR?"  Part="1"
-F 0 "#PWR?" H 1650 2850 50  0001 C CNN
+AR Path="/60084FF3/600A49FC/6008C2BE" Ref="#PWR021"  Part="1"
+F 0 "#PWR021" H 1650 2850 50  0001 C CNN
 F 1 "GND" H 1655 2927 50  0000 C CNN
 F 2 "" H 1650 3100 50  0001 C CNN
@@
 P 3200 2650
 AR Path="/6008501D/6008D2A4" Ref="#PWR?"  Part="1"
-AR Path="/60084FF3/600A49FC/6008D2A4" Ref="#PWR?"  Part="1"
-F 0 "#PWR?" H 3200 2400 50  0001 C CNN
+AR Path="/60084FF3/600A49FC/6008D2A4" Ref="#PWR024"  Part="1"
+F 0 "#PWR024" H 3200 2400 50  0001 C CNN
 F 1 "GND" V 3205 2522 50  0000 R CNN
 F 2 "" H 3200 2650 50  0001 C CNN
@@
 P 5000 2150
 AR Path="/6008501D/60090735" Ref="R?"  Part="1"
-AR Path="/60084FF3/600A49FC/60090735" Ref="R?"  Part="1"
-F 0 "R?" V 4900 2150 50  0000 C CNN
+AR Path="/60084FF3/600A49FC/60090735" Ref="R14"  Part="1"
+F 0 "R14" V 4900 2150 50  0000 C CNN
 F 1 "22" V 5100 2150 50  0000 C CNN
 F 2 "Resistor_SMD:R_0603_1608Metric" V 4930 2150 50  0001 C CNN
 F 3 "~" H 5000 2150 50  0001 C CNN
+F 4 "MOUNT" H 5000 2150 50  0001 C CNN "Mount"
+F 5 "SMD" H 5000 2150 50  0001 C CNN "MountType"
+F 6 "-" H 5000 2150 50  0001 C CNN "Manufacturer"
 	1    5000 2150
 	0    1    1    0
@@
 P 5000 3150
 AR Path="/6008501D/60090CC5" Ref="R?"  Part="1"
-AR Path="/60084FF3/600A49FC/60090CC5" Ref="R?"  Part="1"
-F 0 "R?" V 4900 3150 50  0000 C CNN
+AR Path="/60084FF3/600A49FC/60090CC5" Ref="R15"  Part="1"
+F 0 "R15" V 4900 3150 50  0000 C CNN
 F 1 "22" V 5100 3150 50  0000 C CNN
 F 2 "Resistor_SMD:R_0603_1608Metric" V 4930 3150 50  0001 C CNN
 F 3 "~" H 5000 3150 50  0001 C CNN
+F 4 "MOUNT" H 5000 3150 50  0001 C CNN "Mount"
+F 5 "SMD" H 5000 3150 50  0001 C CNN "MountType"
+F 6 "-" H 5000 3150 50  0001 C CNN "Manufacturer"
 	1    5000 3150
 	0    1    1    0
@@
 P 5000 1800
 AR Path="/6008501D/600911C9" Ref="R?"  Part="1"
-AR Path="/60084FF3/600A49FC/600911C9" Ref="R?"  Part="1"
-F 0 "R?" V 4900 1800 50  0000 C CNN
+AR Path="/60084FF3/600A49FC/600911C9" Ref="R13"  Part="1"
+F 0 "R13" V 4900 1800 50  0000 C CNN
 F 1 "1.5k" V 5100 1800 50  0000 C CNN
 F 2 "Resistor_SMD:R_0603_1608Metric" V 4930 1800 50  0001 C CNN
 F 3 "~" H 5000 1800 50  0001 C CNN
+F 4 "MOUNT" H 5000 1800 50  0001 C CNN "Mount"
+F 5 "SMD" H 5000 1800 50  0001 C CNN "MountType"
+F 6 "-" H 5000 1800 50  0001 C CNN "Manufacturer"
 	1    5000 1800
 	0    1    1    0
@@
 P 2450 3900
 AR Path="/6008501D/600924D4" Ref="#PWR?"  Part="1"
-AR Path="/60084FF3/600A49FC/600924D4" Ref="#PWR?"  Part="1"
-F 0 "#PWR?" H 2450 3650 50  0001 C CNN
+AR Path="/60084FF3/600A49FC/600924D4" Ref="#PWR023"  Part="1"
+F 0 "#PWR023" H 2450 3650 50  0001 C CNN
 F 1 "GND" H 2455 3727 50  0000 C CNN
 F 2 "" H 2450 3900 50  0001 C CNN
@@
 P 2450 3150
 AR Path="/6008501D/60092867" Ref="R?"  Part="1"
-AR Path="/60084FF3/600A49FC/60092867" Ref="R?"  Part="1"
-F 0 "R?" H 2380 3104 50  0000 R CNN
+AR Path="/60084FF3/600A49FC/60092867" Ref="R11"  Part="1"
+F 0 "R11" H 2380 3104 50  0000 R CNN
 F 1 "4.7k" H 2380 3195 50  0000 R CNN
 F 2 "Resistor_SMD:R_0603_1608Metric" V 2380 3150 50  0001 C CNN
-F 3 "~" H 2450 3150 50  0001 C CNN
+F 3 "https://datasheet.lcsc.com/szlcsc/YAGEO-RC0603FR-074K7L_C99782.pdf" H 2450 3150 50  0001 C CNN
+F 4 "MOUNT" H 2450 3150 50  0001 C CNN "Mount"
+F 5 "SMD" H 2450 3150 50  0001 C CNN "MountType"
+F 6 "YAGEO" H 2450 3150 50  0001 C CNN "Manufacturer"
+F 7 "4.7kΩ ±1% 0.1W ±100ppm/℃ 0603 Chip Resistor - Surface Mount RoHS" H 2450 3150 50  0001 C CNN "Description"
+F 8 "RC0603FR-074K7L" H 2450 3150 50  0001 C CNN "PartNumber"
 	1    2450 3150
 	-1   0    0    1
@@
 P 2450 3650
 AR Path="/6008501D/60092D30" Ref="R?"  Part="1"
-AR Path="/60084FF3/600A49FC/60092D30" Ref="R?"  Part="1"
-F 0 "R?" H 2380 3604 50  0000 R CNN
+AR Path="/60084FF3/600A49FC/60092D30" Ref="R12"  Part="1"
+F 0 "R12" H 2380 3604 50  0000 R CNN
 F 1 "10k" H 2380 3695 50  0000 R CNN
 F 2 "Resistor_SMD:R_0603_1608Metric" V 2380 3650 50  0001 C CNN
 F 3 "~" H 2450 3650 50  0001 C CNN
+F 4 "MOUNT" H 2450 3650 50  0001 C CNN "Mount"
+F 5 "SMD" H 2450 3650 50  0001 C CNN "MountType"
+F 6 "-" H 2450 3650 50  0001 C CNN "Manufacturer"
 	1    2450 3650
 	-1   0    0    1
@@
 P 2450 2100
 AR Path="/6008501D/60096CE7" Ref="#PWR?"  Part="1"
-AR Path="/60084FF3/600A49FC/60096CE7" Ref="#PWR?"  Part="1"
-F 0 "#PWR?" H 2450 1950 50  0001 C CNN
+AR Path="/60084FF3/600A49FC/60096CE7" Ref="#PWR022"  Part="1"
+F 0 "#PWR022" H 2450 1950 50  0001 C CNN
 F 1 "+5V" H 2465 2273 50  0000 C CNN
 F 2 "" H 2450 2100 50  0001 C CNN
@@
 P 2100 3400
 AR Path="/6008501D/600A069F" Ref="C?"  Part="1"
-AR Path="/60084FF3/600A49FC/600A069F" Ref="C?"  Part="1"
-F 0 "C?" H 2215 3446 50  0000 L CNN
+AR Path="/60084FF3/600A49FC/600A069F" Ref="C10"  Part="1"
+F 0 "C10" H 2215 3446 50  0000 L CNN
 F 1 "10uF" H 2215 3355 50  0000 L CNN
-F 2 "" H 2138 3250 50  0001 C CNN
-F 3 "~" H 2100 3400 50  0001 C CNN
+F 2 "Capacitor_SMD:C_0805_2012Metric" H 2138 3250 50  0001 C CNN
+F 3 "https://datasheet.lcsc.com/szlcsc/Samsung-Electro-Mechanics-CL21A106KPFNNNE_C17024.pdf" H 2100 3400 50  0001 C CNN
+F 4 "MOUNT" H 2100 3400 50  0001 C CNN "Mount"
+F 5 "SMD" H 2100 3400 50  0001 C CNN "MountType"
+F 6 "Samsung Electro-Mechanics" H 2100 3400 50  0001 C CNN "Manufacturer"
+F 7 "10uF ±10% 10V X5R 0805 Multilayer Ceramic Capacitors MLCC" H 2100 3400 50  0001 C CNN "Description"
+F 8 "CL21A106KPFNNNE" H 2100 3400 50  0001 C CNN "PartNumber"
 	1    2100 3400
 	1    0    0    -1
@@
 P 4300 2650
 AR Path="/6008501D/600A171B" Ref="#PWR?"  Part="1"
-AR Path="/60084FF3/600A49FC/600A171B" Ref="#PWR?"  Part="1"
-F 0 "#PWR?" H 4300 2500 50  0001 C CNN
+AR Path="/60084FF3/600A49FC/600A171B" Ref="#PWR025"  Part="1"
+F 0 "#PWR025" H 4300 2500 50  0001 C CNN
 F 1 "+5V" V 4315 2778 50  0000 L CNN
 F 2 "" H 4300 2650 50  0001 C CNN
@@
 P 5250 2900
 AR Path="/6008501D/600F0CFC" Ref="C?"  Part="1"
-AR Path="/60084FF3/600A49FC/600F0CFC" Ref="C?"  Part="1"
-F 0 "C?" H 5365 2946 50  0000 L CNN
+AR Path="/60084FF3/600A49FC/600F0CFC" Ref="C12"  Part="1"
+F 0 "C12" H 5365 2946 50  0000 L CNN
 F 1 "47p" H 5365 2855 50  0000 L CNN
-F 2 "" H 5288 2750 50  0001 C CNN
-F 3 "~" H 5250 2900 50  0001 C CNN
+F 2 "Capacitor_SMD:C_0603_1608Metric" H 5288 2750 50  0001 C CNN
+F 3 "https://datasheet.lcsc.com/szlcsc/2008261939_Samsung-Electro-Mechanics-CL10C470KB8NNNC_C730450.pdf" H 5250 2900 50  0001 C CNN
+F 4 "MOUNT" H 5250 2900 50  0001 C CNN "Mount"
+F 5 "SMD" H 5250 2900 50  0001 C CNN "MountType"
+F 6 "Samsung Electro-Mechanics" H 5250 2900 50  0001 C CNN "Manufacturer"
+F 7 "47pF ±10% 50V C0G 0603 Multilayer Ceramic Capacitors" H 5250 2900 50  0001 C CNN "Description"
+F 8 "CL10C470KB8NNNC" H 5250 2900 50  0001 C CNN "PartNumber"
 	1    5250 2900
 	1    0    0    -1
@@
 P 5250 2400
 AR Path="/6008501D/600F1442" Ref="C?"  Part="1"
-AR Path="/60084FF3/600A49FC/600F1442" Ref="C?"  Part="1"
-F 0 "C?" H 5365 2446 50  0000 L CNN
+AR Path="/60084FF3/600A49FC/600F1442" Ref="C11"  Part="1"
+F 0 "C11" H 5365 2446 50  0000 L CNN
 F 1 "47p" H 5365 2355 50  0000 L CNN
-F 2 "" H 5288 2250 50  0001 C CNN
-F 3 "~" H 5250 2400 50  0001 C CNN
+F 2 "Capacitor_SMD:C_0603_1608Metric" H 5288 2250 50  0001 C CNN
+F 3 "https://datasheet.lcsc.com/szlcsc/2008261939_Samsung-Electro-Mechanics-CL10C470KB8NNNC_C730450.pdf" H 5250 2400 50  0001 C CNN
+F 4 "MOUNT" H 5250 2400 50  0001 C CNN "Mount"
+F 5 "SMD" H 5250 2400 50  0001 C CNN "MountType"
+F 6 "Samsung Electro-Mechanics" H 5250 2400 50  0001 C CNN "Manufacturer"
+F 7 "47pF ±10% 50V C0G 0603 Multilayer Ceramic Capacitors" H 5250 2400 50  0001 C CNN "Description"
+F 8 "CL10C470KB8NNNC" H 5250 2400 50  0001 C CNN "PartNumber"
 	1    5250 2400
 	1    0    0    -1
@@
 P 5250 2650
 AR Path="/6008501D/600F2F96" Ref="#PWR?"  Part="1"
-AR Path="/60084FF3/600A49FC/600F2F96" Ref="#PWR?"  Part="1"
-F 0 "#PWR?" H 5250 2400 50  0001 C CNN
+AR Path="/60084FF3/600A49FC/600F2F96" Ref="#PWR026"  Part="1"
+F 0 "#PWR026" H 5250 2400 50  0001 C CNN
 F 1 "GND" V 5255 2522 50  0000 R CNN
 F 2 "" H 5250 2650 50  0001 C CNN

Commit message: Start routing
Parts:
- R12: Description (none) -> 10K ±5% 1/10W ±100ppm/℃ 0603 Chip Resistor - Surface Mount; Manufacturer - -> YAGEO; PartNumber (none) -> RC0603JR-0710KL
- R13: Description (none) -> 1.5kΩ ±1% 0.1W ±100ppm/℃ 0603 Chip Resistor - Surface Mount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; Manufacturer - -> YAGEO; PartNumber (none) -> RC0603FR-071K5L
- R14, R15: Description (none) -> 22 ±1% 1/10W ±100ppm/°C 0603 Chip Resistor - Surface Mount; Manufacturer - -> YAGEO; PartNumber (none) -> RC0603FR-0722RL
Changed lines of the file:
@@
 F 1 "22" V 5100 2150 50  0000 C CNN
 F 2 "Resistor_SMD:R_0603_1608Metric" V 4930 2150 50  0001 C CNN
-F 3 "~" H 5000 2150 50  0001 C CNN
+F 3 "https://datasheet.lcsc.com/szlcsc/1809152003_YAGEO-RC0603FR-0722RL_C107701.pdf" H 5000 2150 50  0001 C CNN
 F 4 "MOUNT" H 5000 2150 50  0001 C CNN "Mount"
 F 5 "SMD" H 5000 2150 50  0001 C CNN "MountType"
-F 6 "-" H 5000 2150 50  0001 C CNN "Manufacturer"
+F 6 "YAGEO" H 5000 2150 50  0001 C CNN "Manufacturer"
+F 7 "22 ±1% 1/10W ±100ppm/°C 0603 Chip Resistor - Surface Mount" H 5000 2150 50  0001 C CNN "Description"
+F 8 "RC0603FR-0722RL" H 5000 2150 50  0001 C CNN "PartNumber"
 	1    5000 2150
 	0    1    1    0
@@
 F 1 "22" V 5100 3150 50  0000 C CNN
 F 2 "Resistor_SMD:R_0603_1608Metric" V 4930 3150 50  0001 C CNN
-F 3 "~" H 5000 3150 50  0001 C CNN
+F 3 "https://datasheet.lcsc.com/szlcsc/1809152003_YAGEO-RC0603FR-0722RL_C107701.pdf" H 5000 3150 50  0001 C CNN
 F 4 "MOUNT" H 5000 3150 50  0001 C CNN "Mount"
 F 5 "SMD" H 5000 3150 50  0001 C CNN "MountType"
-F 6 "-" H 5000 3150 50  0001 C CNN "Manufacturer"
+F 6 "YAGEO" H 5000 3150 50  0001 C CNN "Manufacturer"
+F 7 "22 ±1% 1/10W ±100ppm/°C 0603 Chip Resistor - Surface Mount" H 5000 3150 50  0001 C CNN "Description"
+F 8 "RC0603FR-0722RL" H 5000 3150 50  0001 C CNN "PartNumber"
 	1    5000 3150
 	0    1    1    0
@@
 F 1 "1.5k" V 5100 1800 50  0000 C CNN
 F 2 "Resistor_SMD:R_0603_1608Metric" V 4930 1800 50  0001 C CNN
-F 3 "~" H 5000 1800 50  0001 C CNN
+F 3 "https://datasheet.lcsc.com/szlcsc/YAGEO-RC0603FR-071K5L_C114668.pdf" H 5000 1800 50  0001 C CNN
 F 4 "MOUNT" H 5000 1800 50  0001 C CNN "Mount"
 F 5 "SMD" H 5000 1800 50  0001 C CNN "MountType"
-F 6 "-" H 5000 1800 50  0001 C CNN "Manufacturer"
+F 6 "YAGEO" H 5000 1800 50  0001 C CNN "Manufacturer"
+F 7 "1.5kΩ ±1% 0.1W ±100ppm/℃ 0603 Chip Resistor - Surface Mount RoHS" H 5000 1800 50  0001 C CNN "Description"
+F 8 "RC0603FR-071K5L" H 5000 1800 50  0001 C CNN "PartNumber"
 	1    5000 1800
 	0    1    1    0
@@
 F 1 "10k" H 2380 3695 50  0000 R CNN
 F 2 "Resistor_SMD:R_0603_1608Metric" V 2380 3650 50  0001 C CNN
-F 3 "~" H 2450 3650 50  0001 C CNN
+F 3 "https://datasheet.lcsc.com/szlcsc/1811081617_YAGEO-RC0603JR-0710KL_C99198.pdf" H 2450 3650 50  0001 C CNN
 F 4 "MOUNT" H 2450 3650 50  0001 C CNN "Mount"
 F 5 "SMD" H 2450 3650 50  0001 C CNN "MountType"
-F 6 "-" H 2450 3650 50  0001 C CNN "Manufacturer"
+F 6 "YAGEO" H 2450 3650 50  0001 C CNN "Manufacturer"
+F 7 "10K ±5% 1/10W ±100ppm/℃ 0603 Chip Resistor - Surface Mount" H 2450 3650 50  0001 C CNN "Description"
+F 8 "RC0603JR-0710KL" H 2450 3650 50  0001 C CNN "PartNumber"
 	1    2450 3650
 	-1   0    0    1
