File: CANProxy.kicad_pcb (KiCad board)
At the start: 2 copper layers, 83 parts, among them J1 LEFT, J2 RIGHT, J3 DEBUG, J4 USB_B_Micro, SW1 RST, U1 STM32F105RBTx, U2 USBLC6-2SC6, U3 TJA1020T, U4 TJA1051T-3, U5 TJA1020T, U6 TJA1051T-3, U7 KF50BD-TR, U8 LM3940IMP-3.3

Commit message: Start routing
Parts:
- added D10: 5KP15CA, Diode_THT:D_5KP_P10.16mm_Horizontal, F.Cu at (292.0, 45.0)
- added JP10: SolderJumper_2_Open, Jumper:SolderJumper-2_P1.3mm_Open_RoundedPad1.0x1.5mm, F.Cu at (321.0, 49.3)
- added JP4: SolderJumper_2_Open, Jumper:SolderJumper-2_P1.3mm_Open_RoundedPad1.0x1.5mm, F.Cu at (316.6, 41.2)
- added JP5: SolderJumper_2_Open, Jumper:SolderJumper-2_P1.3mm_Open_RoundedPad1.0x1.5mm, F.Cu at (321.0, 41.2)
- added JP9: SolderJumper_2_Open, Jumper:SolderJumper-2_P1.3mm_Open_RoundedPad1.0x1.5mm, F.Cu at (316.6, 49.3)
- added L1: L_Core_Iron, Inductor_SMD:L_1206_3216Metric, F.Cu at (307.1, 41.1)
- moved U2 124.0 mm to (111.0, 89.0), turned to 90 degrees
- moved J1 124.0 mm to (71.0, 78.0), turned to 270 degrees
- moved C12 122.7 mm to (114.0, 84.2), turned to 90 degrees
- moved C11 122.6 mm to (108.0, 84.2), turned to 270 degrees
- moved R15 121.1 mm to (112.0, 84.2), turned to 270 degrees
- moved J4 119.1 mm to (110.0, 96.0)
- moved R14 116.8 mm to (110.0, 84.2), turned to 270 degrees
- moved J3 103.3 mm to (96.0, 32.0), turned to 90 degrees
- moved U1 90.1 mm to (99.0, 49.0)
- moved J2 84.0 mm to (151.0, 95.0), turned to 90 degrees
- renumbered D10 to D11
Connections:
- D11 pad 1: Net-(D10-Pad1) (its old number) -> Net-(C23-Pad1)
- D11 pad 2: ECU -> Net-(D11-Pad2)
- F1 pad 2: Net-(D10-Pad1) (its old number) -> ECU

Commit message: CAN part routing
Parts:
- removed the C15 at (261.1, 42.3)
- removed the C18 at (269.4, 27.9)
- removed the C26 at (249.8, 18.0)
- added C13: 100nF, Capacitor_SMD:C_0603_1608Metric, F.Cu at (92.5, 63.6)
- added C16: 4.7nF, Capacitor_SMD:C_0603_1608Metric, F.Cu at (129.6, 63.5)
- added C20: 220pF, Capacitor_SMD:C_0603_1608Metric, F.Cu at (136.4, 74.7)
- added C21: 1nF, Capacitor_SMD:C_0603_1608Metric, F.Cu at (132.8, 74.7)
- added C28: 47uF, Capacitor_SMD:C_0805_2012Metric, F.Cu at (249.8, 18.0)
- added FB1: BLM18BD102SH1, Inductor_SMD:L_0603_1608Metric, F.Cu at (82.3, 66.0)
- added FB2: BLM18BD102SH1, Inductor_SMD:L_0603_1608Metric, F.Cu at (151.6, 79.0)
- C19: value 1nF -> 100nF
- D5, D8: value SM712-02HTG -> PESD1LIN; footprint Package_TO_SOT_SMD:SOT-23 -> Diode_SMD:D_SOD-323
- D6, D9: value SM712-02HTG -> PESD1CAN
- J4, JP10, JP4, JP5, JP9: moved to B.Cu
- JP1, JP2, JP3, JP6, JP7, JP8: footprint Connector_PinHeader_2.54mm:PinHeader_1x02_P2.54mm_Vertical -> Jumper:SolderJumper-2_P1.3mm_Open_RoundedPad1.0x1.5mm; moved to B.Cu
- moved JP10 231.8 mm to (90.5, 74.4), turned to 180 degrees
- moved JP9 227.1 mm to (90.5, 71.3), turned to 180 degrees
- moved JP5 192.3 mm to (130.2, 65.7)
- moved JP4 188.4 mm to (130.2, 68.8)
- moved D9 183.4 mm to (79.4, 72.8), turned to 180 degrees
- moved C23 178.4 mm to (83.2, 69.8)
- moved R23 175.8 mm to (87.0, 76.4), turned to 180 degrees
- moved C24 173.4 mm to (83.2, 75.9)
- moved FL2 172.6 mm to (85.0, 72.8), turned to 90 degrees
- moved C22 162.4 mm to (90.3, 76.4)
- moved R22 161.0 mm to (86.9, 69.3), turned to 180 degrees
- moved U6 156.8 mm to (94.1, 72.8), turned to 180 degrees
- moved JP1 153.4 mm to (87.4, 66.0), turned to 90 degrees
- moved JP2 151.3 mm to (84.8, 66.0), turned to 90 degrees
- moved JP7 150.8 mm to (132.3, 73.9), turned to 270 degrees
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- renumbered C13 to C14, C14 to C15, C16 to C17, C17 to C18, C20 to C22, C21 to C23, C22 to C24, C23 to C25, C24 to C26, C25 to C27
Connections:
- C19 pad 1: Net-(C19-Pad1) -> ~WAKE
- D4 pad 2: Net-(D4-Pad2) -> ECU
- D5 pad 1: Net-(D5-Pad1) -> LIN1
- D5 pad 2: LIN1 -> GND
- D7 pad 2: Net-(D7-Pad2) -> ECU
- D8 pad 1: Net-(D8-Pad1) -> LIN2
- D8 pad 2: LIN2 -> GND
- F1 pad 2: ECU -> GND
- J1 pad 5: LIN1 -> LIN2
- J2 pad 1: ECU -> GND
- J2 pad 2: CAN2_H -> LIN1
- J2 pad 4: GND -> CAN2_H
- J2 pad 5: LIN2 -> GND
- J2 pad 6: GND -> ECU
- JP1 pad 1: LIN1 -> Net-(FB1-Pad2)
- JP2 pad 1: LIN1 -> Net-(FB1-Pad2)
- JP3 pad 2: LIN1 -> Net-(FB1-Pad2)
- JP6 pad 1: LIN2 -> Net-(FB2-Pad2)
- JP7 pad 1: LIN2 -> Net-(FB2-Pad2)
- JP7 pad 2: Net-(C19-Pad1) -> Net-(C21-Pad1)
- JP8 pad 2: LIN2 -> Net-(FB2-Pad2)
- R16 pad 1: +3V3 -> ECU
- R16 pad 2: /CORE/LIN1_RX -> ~WAKE
- R20 pad 1: +3V3 -> ECU
- R20 pad 2: /CORE/LIN2_RX -> ~WAKE
- U1 pad 15: /CORE/~LIN1_SLP -> Net-(U1-Pad15)
- U1 pad 16: /CORE/LIN1_TX -> Net-(U1-Pad16)
- U1 pad 17: /CORE/LIN1_RX -> Net-(U1-Pad17)
- U1 pad 2: Net-(U1-Pad2) -> /CORE/CAN1_STB
- U1 pad 28: Net-(U1-Pad28) -> /CORE/~LIN1_SLP
- U1 pad 29: /CORE/CAN1_STB -> /CORE/LIN1_TX
- U1 pad 30: Net-(U1-Pad30) -> /CORE/LIN1_RX
- U3 pad 3: Net-(U3-Pad3) -> ~WAKE
- U3 pad 6: LIN1 -> Net-(FB1-Pad2)
- U3 pad 8: Net-(D4-Pad2) -> Net-(U3-Pad8)
- U5 pad 3: Net-(U5-Pad3) -> ~WAKE
- U5 pad 6: LIN2 -> Net-(FB2-Pad2)
- U5 pad 8: Net-(D7-Pad2) -> Net-(U5-Pad8)
Routing:
- net Net-(FB2-Pad2): track 0.00 -> 19.6 mm, vias 0 -> 2
- net +3V3: track 0.00 -> 14.2 mm
- net Net-(C16-Pad1): track 0.00 -> 13.6 mm
- net Net-(C22-Pad1): track 0.00 -> 13.5 mm
- net ECU: track 0.00 -> 12.8 mm, vias 0 -> 2
- net Net-(FB1-Pad2): track 0.00 -> 10.3 mm, vias 0 -> 2
- net HFQ1: track 0.00 -> 10.1 mm
- net Net-(FL2-Pad1): track 0.00 -> 9.49 mm, vias 0 -> 1
- net Net-(FL2-Pad2): track 0.00 -> 9.49 mm, vias 0 -> 1
- net Net-(FL1-Pad1): track 0.00 -> 8.91 mm, vias 0 -> 1
- net Net-(FL1-Pad2): track 0.00 -> 8.54 mm, vias 0 -> 1
- net Net-(D4-Pad1): track 0.00 -> 6.86 mm
- net ~WAKE: track 0.00 -> 6.28 mm
- net Net-(D7-Pad2): track 0.00 -> 5.07 mm
- net CAN1_H: track 0.00 -> 4.67 mm
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